File: schematics-w-display/schematic.kicad_pcb (KiCad board)
At the start: 2 copper layers, 61 x 76.3 mm, 8 parts, among them J1 Conn_01x21_Female, J2 Conn_01x06_Female, J3 Conn_01x21_Female, J4 Conn_01x08_Female

Commit message: Version 2
Parts:
- moved J2 25.5 mm to (92.5, 67.9), turned to 0 degrees
- moved   18.2 mm to (100.2, 90.5)
- moved   18.2 mm to (100.2, 118.5)
- moved   18.2 mm to (143.2, 118.5)
- moved   18.2 mm to (143.2, 90.5)
- moved J4 18.2 mm to (90.2, 112.2)
Routing:
- net /SCL: track 34.6 -> 18.1 mm
- net /BUSY: track 34.5 -> 20.2 mm
- net /RST: track 33.9 -> 20.5 mm
- net /SDA: track 30.5 -> 17.8 mm
- net /DC: track 33.2 -> 20.7 mm
- net /CSB: track 26.1 -> 17.6 mm
- net /CS: track 27.5 -> 21.1 mm
- net /CLK: track 27.1 -> 21.2 mm
- net /MOSI: track 26.9 -> 21.4 mm
- net /SDO: track 21.7 -> 18.9 mm
- net /3v3: track 52.7 -> 51.3 mm
Other:
- board size 61 x 76.3 mm -> 61 x 64.9 mm

Commit message: v3
Parts:
- moved J1 2.00 mm to (135.0, 69.9)
- moved J3 2.00 mm to (110.0, 120.7)
Routing:
- net /CS: track 21.1 -> 20.1 mm
- net /DC: track 20.7 -> 19.9 mm
- net /3v3: track 51.3 -> 52.1 mm
- net /CSB: track 17.6 -> 18.3 mm
- net /MOSI: track 21.4 -> 20.6 mm
- net /SDA: track 17.8 -> 18.3 mm
- net /SDO: track 18.9 -> 18.3 mm
- net /RST: track 20.5 -> 20.0 mm
Other:
- board size 61 x 64.9 mm -> 61 x 63.1 mm
Changed lines of the file:
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@@
     (thickness 1.6)
     (drawings 5)
-    (tracks 45)
+    (tracks 43)
     (zones 0)
     (modules 8)
@@
   )
   (module Connector_PinHeader_2.54mm:PinHeader_1x21_P2.54mm_Vertical (layer F.Cu)
-    (at 135 67.945)
+    (at 135 69.945)
     (descr "Through hole straight pin header, 1x21, 2.54mm pitch, single row")
     (tags "Through hole pin header THT 1x21 2.54mm single row")
@@
   )
   (module Connector_PinHeader_2.54mm:PinHeader_1x21_P2.54mm_Vertical (layer F.Cu)
-    (at 110 118.745 180)
+    (at 110 120.745 180)
     (descr "Through hole straight pin header, 1x21, 2.54mm pitch, single row")
     (tags "Through hole pin header THT 1x21 2.54mm single row")
@@
     (arrow2b (pts (xy 155.700399 90.5) (xy 156.28682 91.626504)))
   )
-  (gr_line (start 147.9 58.2) (end 86.9 58.2) (layer Edge.Cuts) (width 0.05))
-  (gr_line (start 86.9 58.2) (end 86.9 123.063) (layer Edge.Cuts) (width 0.05))
-  (gr_line (start 147.9 123.079) (end 147.9 58.2) (layer Edge.Cuts) (width 0.05))
-  (segment (start 109.955 67.9) (end 110 67.945) (width 0.75) (layer B.Cu) (net 1))
-  (segment (start 103.8 67.9) (end 109.955 67.9) (width 0.75) (layer B.Cu) (net 1))
+  (gr_line (start 147.9 60) (end 86.9 60) (layer Edge.Cuts) (width 0.05))
+  (gr_line (start 86.9 60) (end 86.9 123.063) (layer Edge.Cuts) (width 0.05))
+  (gr_line (start 147.9 123.079) (end 147.9 60) (layer Edge.Cuts) (width 0.05))
   (segment (start 92.5 67.9) (end 94.8 67.9) (width 0.75) (layer B.Cu) (net 1))
   (segment (start 94.8 67.9) (end 94.6 67.9) (width 0.75) (layer B.Cu) (net 1))
-  (segment (start 103.8 67.9) (end 94.8 67.9) (width 0.75) (layer B.Cu) (net 1))
   (segment (start 88.6 96.6) (end 90.2 98.2) (width 0.75) (layer B.Cu) (net 1))
   (segment (start 88.6 70.1) (end 88.6 96.6) (width 0.75) (layer B.Cu) (net 1))
   (segment (start 90.8 67.9) (end 88.6 70.1) (width 0.75) (layer B.Cu) (net 1))
   (segment (start 92.5 67.9) (end 90.8 67.9) (width 0.75) (layer B.Cu) (net 1))
-  (segment (start 109.955 72.98) (end 110 73.025) (width 0.75) (layer B.Cu) (net 2))
-  (segment (start 92.5 72.98) (end 105.18 72.98) (width 0.75) (layer B.Cu) (net 2))
-  (segment (start 105.18 72.98) (end 109.955 72.98) (width 0.75) (layer B.Cu) (net 2))
-  (segment (start 103.8 72.98) (end 105.18 72.98) (width 0.75) (layer B.Cu) (net 2))
-  (segment (start 109.955 75.52) (end 110 75.565) (width 0.75) (layer B.Cu) (net 3))
-  (segment (start 92.5 75.52) (end 103.88 75.52) (width 0.75) (layer B.Cu) (net 3))
-  (segment (start 103.88 75.52) (end 109.955 75.52) (width 0.75) (layer B.Cu) (net 3))
-  (segment (start 103.8 75.52) (end 103.88 75.52) (width 0.75) (layer B.Cu) (net 3))
-  (segment (start 109.955 78.06) (end 110 78.105) (width 0.75) (layer B.Cu) (net 4))
-  (segment (start 92.5 78.06) (end 104.04 78.06) (width 0.75) (layer B.Cu) (net 4))
-  (segment (start 104.04 78.06) (end 109.955 78.06) (width 0.75) (layer B.Cu) (net 4))
-  (segment (start 103.8 78.06) (end 104.04 78.06) (width 0.75) (layer B.Cu) (net 4))
-  (segment (start 109.955 80.6) (end 110 80.645) (width 0.75) (layer B.Cu) (net 5))
-  (segment (start 103.8 80.6) (end 109.955 80.6) (width 0.75) (layer B.Cu) (net 5))
-  (segment (start 92.5 80.6) (end 104.4 80.6) (width 0.75) (layer B.Cu) (net 5))
+  (segment (start 107.955 67.9) (end 110 69.945) (width 0.75) (layer B.Cu) (net 1))
+  (segment (start 94.8 67.9) (end 107.955 67.9) (width 0.75) (layer B.Cu) (net 1))
+  (segment (start 92.5 72.98) (end 104.38 72.98) (width 0.75) (layer B.Cu) (net 2))
+  (segment (start 104.38 72.98) (end 106.425 75.025) (width 0.75) (layer B.Cu) (net 2))
+  (segment (start 108.525 75.025) (end 110 75.025) (width 0.75) (layer B.Cu) (net 2))
+  (segment (start 106.425 75.025) (end 108.525 75.025) (width 0.75) (layer B.Cu) (net 2))
+  (segment (start 103.8 75.52) (end 105.845 77.565) (width 0.75) (layer B.Cu) (net 3))
+  (segment (start 92.5 75.52) (end 103.8 75.52) (width 0.75) (layer B.Cu) (net 3))
+  (segment (start 107.765 77.565) (end 110 77.565) (width 0.75) (layer B.Cu) (net 3))
+  (segment (start 105.845 77.565) (end 107.765 77.565) (width 0.75) (layer B.Cu) (net 3))
+  (segment (start 92.5 78.06) (end 102.16 78.06) (width 0.75) (layer B.Cu) (net 4))
+  (segment (start 102.16 78.06) (end 104.205 80.105) (width 0.75) (layer B.Cu) (net 4))
+  (segment (start 107.795 80.105) (end 110 80.105) (width 0.75) (layer B.Cu) (net 4))
+  (segment (start 104.205 80.105) (end 107.795 80.105) (width 0.75) (layer B.Cu) (net 4))
+  (segment (start 92.5 80.6) (end 100.8 80.6) (width 0.75) (layer B.Cu) (net 5))
+  (segment (start 102.845 82.645) (end 110 82.645) (width 0.75) (layer B.Cu) (net 5))
+  (segment (start 100.8 80.6) (end 102.845 82.645) (width 0.75) (layer B.Cu) (net 5))
   (segment (start 90.2 102.2) (end 93.4 102.2) (width 0.75) (layer B.Cu) (net 7))
-  (segment (start 93.4 102.2) (end 97 98.6) (width 0.75) (layer B.Cu) (net 7))
-  (segment (start 109.825 98.6) (end 110 98.425) (width 0.75) (layer B.Cu) (net 7))
-  (segment (start 97 98.6) (end 109.825 98.6) (width 0.75) (layer B.Cu) (net 7))
-  (segment (start 109.935 100.9) (end 110 100.965) (width 0.75) (layer B.Cu) (net 8))
-  (segment (start 95.2 104.2) (end 98.435 100.965) (width 0.75) (layer B.Cu) (net 8))
-  (segment (start 98.435 100.965) (end 110 100.965) (width 0.75) (layer B.Cu) (net 8))
-  (segment (start 90.2 104.2) (end 95.2 104.2) (width 0.75) (layer B.Cu) (net 8))
-  (segment (start 109.905 103.6) (end 110 103.505) (width 0.75) (layer B.Cu) (net 9))
-  (segment (start 99.895 103.505) (end 110 103.505) (width 0.75) (layer B.Cu) (net 9))
-  (segment (start 97.2 106.2) (end 99.895 103.505) (width 0.75) (layer B.Cu) (net 9))
-  (segment (start 90.2 106.2) (end 97.2 106.2) (width 0.75) (layer B.Cu) (net 9))
-  (segment (start 90.2 108.2) (end 99 108.2) (width 0.75) (layer B.Cu) (net 10))
-  (segment (start 101.155 106.045) (end 110 106.045) (width 0.75) (layer B.Cu) (net 10))
-  (segment (start 99 108.2) (end 101.155 106.045) (width 0.75) (layer B.Cu) (net 10))
-  (segment (start 90.2 110.2) (end 101 110.2) (width 0.75) (layer B.Cu) (net 11))
-  (segment (start 102.615 108.585) (end 110 108.585) (width 0.75) (layer B.Cu) (net 11))
-  (segment (start 101 110.2) (end 102.615 108.585) (width 0.75) (layer B.Cu) (net 11))
-  (segment (start 90.2 112.2) (end 103.4 112.2) (width 0.75) (layer B.Cu) (net 12))
-  (segment (start 104.475 111.125) (end 110 111.125) (width 0.75) (layer B.Cu) (net 12))
-  (segment (start 103.4 112.2) (end 104.475 111.125) (width 0.75) (layer B.Cu) (net 12))
+  (segment (start 109.935 100.9) (end 110 100.965) (width 0.75) (layer B.Cu) (net 7))
+  (segment (start 95.175 100.425) (end 110 100.425) (width 0.75) (layer B.Cu) (net 7))
+  (segment (start 93.4 102.2) (end 95.175 100.425) (width 0.75) (layer B.Cu) (net 7))
+  (segment (start 94.5 104.2) (end 99.8 104.2) (width 0.75) (layer B.Cu) (net 8))
+  (segment (start 90.2 104.2) (end 94.5 104.2) (width 0.75) (layer B.Cu) (net 8))
+  (segment (start 94.5 104.2) (end 95.2 104.2) (width 0.75) (layer B.Cu) (net 8))
+  (segment (start 101.035 102.965) (end 110 102.965) (width 0.75) (layer B.Cu) (net 8))
+  (segment (start 99.8 104.2) (end 101.035 102.965) (width 0.75) (layer B.Cu) (net 8))
+  (segment (start 105.395 105.505) (end 110 105.505) (width 0.75) (layer B.Cu) (net 9))
+  (segment (start 104.7 106.2) (end 105.395 105.505) (width 0.75) (layer B.Cu) (net 9))
+  (segment (start 90.2 106.2) (end 104.7 106.2) (width 0.75) (layer B.Cu) (net 9))
+  (segment (start 109.845 108.2) (end 110 108.045) (width 0.75) (layer B.Cu) (net 10))
+  (segment (start 90.2 108.2) (end 109.845 108.2) (width 0.75) (layer B.Cu) (net 10))
+  (segment (start 104.685 110.585) (end 110 110.585) (width 0.75) (layer B.Cu) (net 11))
+  (segment (start 104.3 110.2) (end 104.685 110.585) (width 0.75) (layer B.Cu) (net 11))
+  (segment (start 90.2 110.2) (end 104.3 110.2) (width 0.75) (layer B.Cu) (net 11))
+  (segment (start 104.825 113.125) (end 110 113.125) (width 0.75) (layer B.Cu) (net 12))
+  (segment (start 103.9 112.2) (end 104.825 113.125) (width 0.75) (layer B.Cu) (net 12))
+  (segment (start 90.2 112.2) (end 103.9 112.2) (width 0.75) (layer B.Cu) (net 12))
   (zone (net 6) (net_name GND) (layer B.Cu) (hatch edge 0.508)
     (connect_pads (clearance 0.508))
@@
     (polygon
       (pts
-        (xy 146.9 122.1) (xy 87.8 122.1) (xy 87.7 59.1) (xy 146.9 59.1)
+        (xy 147.4 122.5) (xy 87.4 122.6) (xy 87.5 60.6) (xy 147.5 60.6)
       )
     )

Commit message: v4
Parts:
- moved   0.50 mm to (99.7, 90.5)
- moved   0.50 mm to (99.7, 118.5)
- moved   0.50 mm to (142.7, 118.5)
- moved   0.50 mm to (142.7, 90.5)
- moved J1 0.50 mm to (135.0, 70.4)
- moved J3 0.50 mm to (110.0, 121.2)
- moved J4 0.50 mm to (89.7, 112.2)
Routing:
- net /RST: track 20.0 -> 21.0 mm
- net /BUSY: track 20.2 -> 20.9 mm
Other:
- board size 61 x 63.1 mm -> 59.8 x 62 mm

Commit message: Final version
Other:
- board size 59.8 x 62 mm -> 59.8 x 61.5 mm
Changed lines of the file:
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@@
   )
   (gr_line (start 87.1 123.063) (end 146.9 123.079) (layer Edge.Cuts) (width 0.05))
-  (gr_line (start 146.9 61.1) (end 87.1 61.1) (layer Edge.Cuts) (width 0.05))
-  (gr_line (start 87.1 61.1) (end 87.1 123.063) (layer Edge.Cuts) (width 0.05))
-  (gr_line (start 146.9 123.079) (end 146.9 61.1) (layer Edge.Cuts) (width 0.05))
+  (gr_line (start 146.9 61.6) (end 87.1 61.6) (layer Edge.Cuts) (width 0.05))
+  (gr_line (start 87.1 61.6) (end 87.1 123.063) (layer Edge.Cuts) (width 0.05))
+  (gr_line (start 146.9 123.079) (end 146.9 61.6) (layer Edge.Cuts) (width 0.05))
   (segment (start 92.5 67.9) (end 94.8 67.9) (width 0.75) (layer B.Cu) (net 1))
   (segment (start 94.8 67.9) (end 94.6 67.9) (width 0.75) (layer B.Cu) (net 1))
@@
     (polygon
       (pts
-        (xy 146.3 122.5) (xy 87.7 122.5) (xy 87.65 61.6) (xy 146.3 61.7)
+        (xy 146.4 122.5) (xy 87.7 122.5) (xy 87.6 62.1) (xy 146.4 62.1)
       )
     )

Commit message: Maybe not so final version
Parts:
- J4: footprint Connector_JST:JST_PH_B8B-PH-K_1x08_P2.00mm_Vertical -> Connector_JST:JST_PH_S8B-PH-K_1x08_P2.00mm_Horizontal
- moved J4 21.6 mm to (105.7, 97.7), turned to 270 degrees
Connections:
- J4 pad 1: /BUSY -> /3v3
- J4 pad 2: /RST -> GND
- J4 pad 3: /DC -> /MOSI
- J4 pad 4: /CS -> /CLK
- J4 pad 5: /CLK -> /CS
- J4 pad 6: /MOSI -> /DC
- J4 pad 7: GND -> /RST
- J4 pad 8: /3v3 -> /BUSY
Routing:
- net /CLK: track 20.8 -> 4.40 mm
- net /RST: track 21.0 -> 4.87 mm
- net /BUSY: track 20.9 -> 5.10 mm
- net /MOSI: track 20.4 -> 4.71 mm
- net /DC: track 20.2 -> 4.87 mm
- net /CS: track 19.9 -> 4.70 mm
- net /3v3: track 52.3 -> 66.1 mm

Commit message: Final version: again
Parts:
- moved   3.80 mm to (99.7, 86.7)
- moved   3.80 mm to (99.7, 114.7)
- moved   3.80 mm to (142.7, 114.7)
- moved   3.80 mm to (142.7, 86.7)
- moved J4 3.00 mm to (105.7, 94.7)
Routing:
- net /3v3: track 66.1 -> 61.2 mm
- net /RST: track 4.87 -> 7.91 mm
- net /BUSY: track 5.10 -> 8.04 mm
- net /CS: track 4.70 -> 7.43 mm
- net /CLK: track 4.40 -> 6.98 mm
- net /DC: track 4.87 -> 6.98 mm
- net /MOSI: track 4.71 -> 6.56 mm
Other:
- outline, holes or cut-outs redrawn
Changed lines of the file:
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@@
   (general
     (thickness 1.6)
-    (drawings 4)
-    (tracks 43)
+    (drawings 9)
+    (tracks 58)
     (zones 0)
     (modules 8)
@@
   )
   (setup
-    (last_trace_width 0.75)
+    (last_trace_width 0.5)
+    (user_trace_width 0.5)
     (user_trace_width 0.75)
     (trace_clearance 0.2)
@@
   )
   (module Connector_JST:JST_PH_S8B-PH-K_1x08_P2.00mm_Horizontal (layer F.Cu)
-    (at 105.7 97.7 270)
+    (at 105.7 94.7 270)
     (descr "JST PH series connector, S8B-PH-K (http://www.jst-mfg.com/product/pdf/eng/ePH.pdf), generated with kicad-footprint-generator")
     (tags "connector JST PH top entry")
@@
   )
   (module MountingHole:MountingHole_3.2mm_M3 (layer F.Cu)
-    (at 99.7 90.5)
+    (at 99.7 86.7)
     (descr "Mounting Hole 3.2mm, no annular, M3")
     (tags "mounting hole 3.2mm no annular m3")
@@
   )
   (module MountingHole:MountingHole_3.2mm_M3 (layer F.Cu)
-    (at 99.7 118.5)
+    (at 99.7 114.7)
     (descr "Mounting Hole 3.2mm, no annular, M3")
     (tags "mounting hole 3.2mm no annular m3")
@@
   )
   (module MountingHole:MountingHole_3.2mm_M3 (layer F.Cu)
-    (at 142.7 118.5)
+    (at 142.7 114.7)
     (descr "Mounting Hole 3.2mm, no annular, M3")
     (tags "mounting hole 3.2mm no annular m3")
@@
   )
   (module MountingHole:MountingHole_3.2mm_M3 (layer F.Cu)
-    (at 142.7 90.5)
+    (at 142.7 86.7)
     (descr "Mounting Hole 3.2mm, no annular, M3")
     (tags "mounting hole 3.2mm no annular m3")
@@
     )
   )
+  (gr_line (start 146.9 72.6) (end 146.9 72.6) (layer Edge.Cuts) (width 0.05))
+  (gr_line (start 146.9 68.6) (end 146.9 61.6) (layer Edge.Cuts) (width 0.05))
+  (gr_line (start 142.9 72.6) (end 146.9 72.6) (layer Edge.Cuts) (width 0.05))
+  (gr_line (start 142.9 68.6) (end 142.9 72.6) (layer Edge.Cuts) (width 0.05))
+  (gr_line (start 146.9 68.6) (end 142.9 68.6) (layer Edge.Cuts) (width 0.05))
   (gr_line (start 87.1 123.063) (end 146.9 123.079) (layer Edge.Cuts) (width 0.05))
   (gr_line (start 146.9 61.6) (end 87.1 61.6) (layer Edge.Cuts) (width 0.05))
   (gr_line (start 87.1 61.6) (end 87.1 123.063) (layer Edge.Cuts) (width 0.05))
-  (gr_line (start 146.9 123.079) (end 146.9 61.6) (layer Edge.Cuts) (width 0.05))
+  (gr_line (start 146.9 123.079) (end 146.9 72.6) (layer Edge.Cuts) (width 0.05))
   (segment (start 92.5 67.9) (end 94.8 67.9) (width 0.75) (layer B.Cu) (net 1))
   (segment (start 94.8 67.9) (end 94.6 67.9) (width 0.75) (layer B.Cu) (net 1))
   (segment (start 107.455 67.9) (end 110 70.445) (width 0.75) (layer B.Cu) (net 1))
   (segment (start 94.8 67.9) (end 107.455 67.9) (width 0.75) (layer B.Cu) (net 1))
+  (segment (start 105.6 94.6) (end 105.7 94.7) (width 0.75) (layer B.Cu) (net 1))
+  (segment (start 94.9 94.6) (end 105.6 94.6) (width 0.75) (layer B.Cu) (net 1))
+  (segment (start 89.3 69) (end 89.3 89) (width 0.75) (layer B.Cu) (net 1))
+  (segment (start 89.3 89) (end 94.9 94.6) (width 0.75) (layer B.Cu) (net 1))
+  (segment (start 90.4 67.9) (end 89.3 69) (width 0.75) (layer B.Cu) (net 1))
   (segment (start 92.5 67.9) (end 90.4 67.9) (width 0.75) (layer B.Cu) (net 1))
-  (segment (start 90.4 67.9) (end 89.3 69) (width 0.75) (layer B.Cu) (net 1))
-  (segment (start 89.3 69) (end 89.3 95.3) (width 0.75) (layer B.Cu) (net 1))
-  (segment (start 91.7 97.7) (end 89.3 95.3) (width 0.75) (layer B.Cu) (net 1))
-  (segment (start 105.7 97.7) (end 91.7 97.7) (width 0.75) (layer B.Cu) (net 1))
   (segment (start 107.425 75.525) (end 110 75.525) (width 0.75) (layer B.Cu) (net 2))
   (segment (start 104.88 72.98) (end 107.425 75.525) (width 0.75) (layer B.Cu) (net 2))
@@
   (segment (start 100.8 80.7) (end 103.245 83.145) (width 0.75) (layer B.Cu) (net 5))
   (segment (start 109.935 100.9) (end 110 100.965) (width 0.75) (layer B.Cu) (net 7))
-  (segment (start 105.7 101.7) (end 107.9 101.7) (width 0.75) (layer B.Cu) (net 7))
-  (segment (start 108.675 100.925) (end 110 100.925) (width 0.75) (layer B.Cu) (net 7))
-  (segment (start 107.9 101.7) (end 108.675 100.925) (width 0.75) (layer B.Cu) (net 7))
-  (segment (start 105.7 103.7) (end 108 103.7) (width 0.75) (layer B.Cu) (net 8))
-  (segment (start 108.235 103.465) (end 110 103.465) (width 0.75) (layer B.Cu) (net 8))
-  (segment (start 108 103.7) (end 108.235 103.465) (width 0.75) (layer B.Cu) (net 8))
+  (segment (start 110 100.925) (end 109.525 100.925) (width 0.75) (layer B.Cu) (net 7))
+  (segment (start 109.225 100.925) (end 110 100.925) (width 0.25) (layer B.Cu) (net 7))
+  (segment (start 105.7 98.7) (end 107.1 98.7) (width 0.5) (layer B.Cu) (net 7))
+  (segment (start 109.325 100.925) (end 110 100.925) (width 0.5) (layer B.Cu) (net 7))
+  (segment (start 107.1 98.7) (end 109.325 100.925) (width 0.5) (layer B.Cu) (net 7))
+  (segment (start 105.7 100.7) (end 106.5 100.7) (width 0.25) (layer B.Cu) (net 8))
+  (segment (start 109.265 103.465) (end 110 103.465) (width 0.25) (layer B.Cu) (net 8))
+  (segment (start 105.7 100.7) (end 106.6 100.7) (width 0.5) (layer B.Cu) (net 8))
+  (segment (start 109.365 103.465) (end 110 103.465) (width 0.5) (layer B.Cu) (net 8))
+  (segment (start 106.6 100.7) (end 109.365 103.465) (width 0.5) (layer B.Cu) (net 8))
   (segment (start 109.805 106.2) (end 110 106.005) (width 0.75) (layer B.Cu) (net 9))
-  (segment (start 105.7 105.7) (end 107.4 105.7) (width 0.75) (layer B.Cu) (net 9))
-  (segment (start 107.705 106.005) (end 110 106.005) (width 0.75) (layer B.Cu) (net 9))
-  (segment (start 107.4 105.7) (end 107.705 106.005) (width 0.75) (layer B.Cu) (net 9))
+  (segment (start 110 106.005) (end 109.605 106.005) (width 0.75) (layer B.Cu) (net 9))
+  (segment (start 105.7 102.7) (end 106.4 102.7) (width 0.25) (layer B.Cu) (net 9))
+  (segment (start 109.705 106.005) (end 110 106.005) (width 0.25) (layer B.Cu) (net 9))
+  (segment (start 109.905 106.005) (end 110 106.005) (width 0.25) (layer B.Cu) (net 9))
+  (segment (start 105.7 102.7) (end 106.2 102.7) (width 0.5) (layer B.Cu) (net 9))
+  (segment (start 109.505 106.005) (end 110 106.005) (width 0.5) (layer B.Cu) (net 9))
+  (segment (start 106.2 102.7) (end 109.505 106.005) (width 0.5) (layer B.Cu) (net 9))
   (segment (start 109.845 108.2) (end 110 108.045) (width 0.75) (layer B.Cu) (net 10))
-  (segment (start 105.7 107.7) (end 106.8 107.7) (width 0.75) (layer B.Cu) (net 10))
-  (segment (start 107.645 108.545) (end 110 108.545) (width 0.75) (layer B.Cu) (net 10))
-  (segment (start 106.8 107.7) (end 107.645 108.545) (width 0.75) (layer B.Cu) (net 10))
-  (segment (start 105.7 109.7) (end 106.9 109.7) (width 0.75) (layer B.Cu) (net 11))
-  (segment (start 108.285 111.085) (end 110 111.085) (width 0.75) (layer B.Cu) (net 11))
-  (segment (start 106.9 109.7) (end 108.285 111.085) (width 0.75) (layer B.Cu) (net 11))
-  (segment (start 105.7 111.7) (end 106.2 111.7) (width 0.75) (layer B.Cu) (net 12))
-  (segment (start 108.125 113.625) (end 110 113.625) (width 0.75) (layer B.Cu) (net 12))
-  (segment (start 106.2 111.7) (end 108.125 113.625) (width 0.75) (layer B.Cu) (net 12))
+  (segment (start 105.7 104.7) (end 106.155 104.7) (width 0.25) (layer B.Cu) (net 10))
+  (segment (start 105.7 104.7) (end 106.2 104.7) (width 0.5) (layer B.Cu) (net 10))
+  (segment (start 106.2 104.7) (end 108.7 107.2) (width 0.5) (layer B.Cu) (net 10))
+  (segment (start 108.7 107.2) (end 108.7 107.9) (width 0.5) (layer B.Cu) (net 10))
+  (segment (start 109.345 108.545) (end 110 108.545) (width 0.5) (layer B.Cu) (net 10))
+  (segment (start 108.7 107.9) (end 109.345 108.545) (width 0.5) (layer B.Cu) (net 10))
+  (segment (start 105.7 106.7) (end 106.2 106.7) (width 0.25) (layer B.Cu) (net 11))
+  (segment (start 105.7 106.7) (end 106.5 106.7) (width 0.25) (layer B.Cu) (net 11))
+  (segment (start 106.2 106.7) (end 107.7 108.2) (width 0.5) (layer B.Cu) (net 11))
+  (segment (start 107.7 108.2) (end 107.7 109.9) (width 0.5) (layer B.Cu) (net 11))
+  (segment (start 108.885 111.085) (end 110 111.085) (width 0.5) (layer B.Cu) (net 11))
+  (segment (start 107.7 109.9) (end 108.885 111.085) (width 0.5) (layer B.Cu) (net 11))
+  (segment (start 105.7 108.7) (end 105.7 111.6) (width 0.5) (layer B.Cu) (net 12))
+  (segment (start 107.725 113.625) (end 110 113.625) (width 0.5) (layer B.Cu) (net 12))
+  (segment (start 105.7 111.6) (end 107.725 113.625) (width 0.5) (layer B.Cu) (net 12))
   (zone (net 6) (net_name GND) (layer B.Cu) (hatch edge 0.508)
     (connect_pads (clearance 0.508))
@@
     (polygon
       (pts
-        (xy 146.4 122.5) (xy 87.7 122.5) (xy 87.6 62.1) (xy 146.4 62.1)
+        (xy 146.4 68.1) (xy 142.4 68.1) (xy 142.4 73.1) (xy 146.4 73.1) (xy 146.4 122.5)
+        (xy 87.7 122.5) (xy 87.6 62.1) (xy 146.4 62.1)
       )
     )
