File: schematics-v2/schematic.sch (KiCad schematic (older format))
At the start: 3 parts, among them J1 Conn_01x21_Female, J2 Conn_01x06_Female, J3 Conn_01x21_Female

Commit message: Some schematic
Parts:
- added SW1: RST_Push, symbol Switch:SW_Push
- added SW2: SW_Push, symbol Switch:SW_Push
Connections:
- net GND: now also SW1.2, SW2.1
- net at J1.2 (Pin_2): now also SW1.1
- net at J3.20 (Pin_20): now also SW2.2
- no-connect marks 35 -> 33
Changed lines of the file:
@@
 NoConn ~ 5250 3400
 NoConn ~ 5250 3300
-NoConn ~ 5250 3200
 NoConn ~ 4400 3800
 NoConn ~ 4400 3700
 NoConn ~ 4400 5000
 NoConn ~ 4400 4900
-NoConn ~ 4400 3200
 NoConn ~ 4400 4800
 NoConn ~ 4400 4700
@@
 Text GLabel 5250 3100 1    50   Input ~ 0
 GND
+$Comp
+L Switch:SW_Push SW1
+U 1 1 6242CDC4
+P 5900 3200
+F 0 "SW1" H 5900 3485 50  0000 C CNN
+F 1 "RST_Push" H 5900 3394 50  0000 C CNN
+F 2 "" H 5900 3400 50  0001 C CNN
+F 3 "~" H 5900 3400 50  0001 C CNN
+	1    5900 3200
+	1    0    0    -1
+$EndComp
+Wire Wire Line
+	5700 3200 5250 3200
+Text GLabel 6100 3200 2    50   Input ~ 0
+GND
+$Comp
+L Switch:SW_Push SW2
+U 1 1 6242FB35
+P 3650 3200
+F 0 "SW2" H 3650 3485 50  0000 C CNN
+F 1 "SW_Push" H 3650 3394 50  0000 C CNN
+F 2 "" H 3650 3400 50  0001 C CNN
+F 3 "~" H 3650 3400 50  0001 C CNN
+	1    3650 3200
+	1    0    0    -1
+$EndComp
+Wire Wire Line
+	3850 3200 4400 3200
+Text GLabel 3450 3200 0    50   Input ~ 0
+GND
 $EndSCHEMATC
